Commit message: nye xacro filer

File: src/qube_description/urdf/qube.macro.xacro (robot description, xacro)
@@ -1,11 +1,21 @@
 <?xml version="1.0"?>
-<robot xmlns:xacro="http://www.ros.org/wiki/xacro" name="joint_model_macro">
-  <xacro:macro name="joint_model" params="prefix">
-        Svart kube fra origo, med ein raud disk på toppen, som har ein kvit viser langs radiusen på overflata.
-    <!-- Stator link: svart boks -->
+<robot xmlns:xacro="http://www.ros.org/wiki/xacro" name="qube_macro">
+  <!-- Parametere -->
+  <xacro:property name="box_size" value="0.102"/>          <!-- Størrelse på den svarte boksen -->
+  <xacro:property name="disk_radius" value="0.025"/>       <!-- Radius for den røde disken -->
+  <xacro:property name="disk_thickness" value="0.01"/>      <!-- Tykkelse på den røde disken -->
+  <xacro:property name="indicator_length" value="0.025"/>   <!-- Lengde på den hvite indikatoren -->
+  <xacro:property name="indicator_width" value="0.002"/>
+  <xacro:property name="indicator_height" value="0.002"/>
+  <!-- Kalkulerte størrelser -->
+  <xacro:property name="half_box_size" value="$(expr ${box_size} / 2)"/>
+  <xacro:property name="disk_z" value="$(expr ${box_size} + ${disk_thickness} / 2)"/>
+  <!-- Makro: 'qube' med valgfritt prefix for gjenbrukbarhet -->
+  <xacro:macro name="qube" params="prefix">
+    <!-- Svarte boksen (stator) -->
     <link name="${prefix}stator_link">
       <visual>
         <geometry>
-          <box size="0.102 0.102 0.102"/>
+          <box size="${box_size} ${box_size} ${box_size}"/>
         </geometry>
         <material name="black">
@@ -14,9 +24,9 @@
       </visual>
     </link>
-    <!-- Rotor link: rød sylinder -->
+    <!-- Røde disken (rotor) -->
     <link name="${prefix}rotor_link">
       <visual>
         <geometry>
-          <cylinder radius="0.025" length="0.01"/>
+          <cylinder radius="${disk_radius}" length="${disk_thickness}"/>
         </geometry>
         <material name="red">
@@ -25,9 +35,9 @@
       </visual>
     </link>
-    <!-- Angle link: hvit boks -->
-    <link name="${prefix}angle_link">
+    <!-- Hvite indikatoren -->
+    <link name="${prefix}indicator_link">
       <visual>
         <geometry>
-          <box size="0.025 0.002 0.002"/>
+          <box size="${indicator_length} ${indicator_width} ${indicator_height}"/>
         </geometry>
         <material name="white">
@@ -36,27 +46,24 @@
       </visual>
     </link>
-    <!-- stator_joint: Fixed joint mellom base_link (definert i hovedfilen) og stator_link -->
+    <!-- Fiksert joint: kobler base_link til den svarte boksen -->
     <joint name="${prefix}stator_joint" type="fixed">
       <parent link="${prefix}base_link"/>
       <child link="${prefix}stator_link"/>
-      <!-- Plasserer stator_link slik at midten (0.102/2 = 0.051 m) ligger over base_link -->
-      <origin xyz="0 0 0.051" rpy="0 0 0"/>
+      <origin xyz="0 0 ${half_box_size}" rpy="0 0 0"/>
     </joint>
-    <!-- angle: Revolute joint mellom stator_link og rotor_link -->
-    <joint name="${prefix}angle" type="revolute">
+    <!-- Revolute joint: disken spinner i forhold til boksen -->
+    <joint name="${prefix}disk_joint" type="revolute">
       <parent link="${prefix}stator_link"/>
       <child link="${prefix}rotor_link"/>
-      <!-- Plasserer rotor_link slik at dens bunn møter toppen av stator_link (0.102 m) -->
-      <origin xyz="0 0 0.053" rpy="0 0 0"/>
+      <origin xyz="0 0 ${disk_z}" rpy="0 0 0"/>
       <axis xyz="0 0 1"/>
-      <limit effort="1.0" velocity="1.0" lower="-3.14" upper="3.14"/>
+      <limit lower="-3.14" upper="3.14" effort="1.0" velocity="1.0"/>
     </joint>
-    <!-- indicator: Fixed joint mellom rotor_link og angle_link -->
-    <joint name="${prefix}indicator" type="fixed">
+    <!-- Fiksert joint: fester den hvite indikatoren til disken -->
+    <joint name="${prefix}indicator_joint" type="fixed">
       <parent link="${prefix}rotor_link"/>
-      <child link="${prefix}angle_link"/>
-      <!-- Plasserer angle_link slik at den stikker ut fra rotoren:
-           Eksempelvis 0.0125 m i x og 0.005 m i z -->
-      <origin xyz="0.0125 0 0.005" rpy="0 0 0"/>
+      <child link="${prefix}indicator_link"/>
+      <!-- Plasserer indikatoren til å stikke ut fra disken (langs x-aksen) -->
+      <origin xyz="${disk_radius} 0 0" rpy="0 0 0"/>
     </joint>
   </xacro:macro>

File: src/qube_description/urdf/qube.urdf.xacro (robot description, xacro)
@@ -1,15 +1,16 @@
 <?xml version="1.0"?>
-<robot name="qube" xmlns:xacro="http://www.ros.org/wiki/xacro">
+<robot xmlns:xacro="http://www.ros.org/wiki/xacro" name="qube_scene">
+  <!-- Inkluder makrofilen -->
   <xacro:include filename="$(find qube_description)/urdf/qube.macro.xacro"/>
-  <xacro:property name="box_width" value="0.102"/>
-  <xacro:property name="angle_link_length" value="0.025"/>
-  <xacro:property name="angle_link_width" value="0.002"/>
+  <!-- Definer world og base_link -->
   <link name="world"/>
   <link name="base_link"/>
-  <joint name="base_joint" type="fixed">
+  <!-- Joint som knytter base_link til world -->
+  <joint name="world_joint" type="fixed">
     <parent link="world"/>
     <child link="base_link"/>
     <origin xyz="0 0 0" rpy="0 0 0"/>
   </joint>
-  <xacro:joint_model prefix=""/>
+  <!-- Instansier Qube-makroen -->
+  <xacro:qube prefix=""/>
 </robot>

Commit message: Sletta test, oppdatert setup, manuelt satt half box disk_z

File: src/qube_description/urdf/qube.macro.xacro (robot description, xacro)
@@ -9,6 +9,6 @@
   <xacro:property name="indicator_height" value="0.002"/>
   <!-- Kalkulerte størrelser -->
-  <xacro:property name="half_box_size" value="$(expr ${box_size} / 2)"/>
-  <xacro:property name="disk_z" value="$(expr ${box_size} + ${disk_thickness} / 2)"/>
+  <xacro:property name="half_box_size" value="0.051"/>
+  <xacro:property name="disk_z" value="0.107"/>
   <!-- Makro: 'qube' med valgfritt prefix for gjenbrukbarhet -->
   <xacro:macro name="qube" params="prefix">

Commit message: sletta driver (error) endra macro, config fil

File: src/qube_description/urdf/qube.macro.xacro (robot description, xacro)
@@ -10,5 +10,5 @@
   <!-- Kalkulerte størrelser -->
   <xacro:property name="half_box_size" value="0.051"/>
-  <xacro:property name="disk_z" value="0.107"/>
+  <xacro:property name="disk_z" value="0.056"/>
   <!-- Makro: 'qube' med valgfritt prefix for gjenbrukbarhet -->
   <xacro:macro name="qube" params="prefix">

Commit message: fikset hvit strek

File: src/qube_description/urdf/qube.macro.xacro (robot description, xacro)
@@ -65,5 +65,5 @@
       <child link="${prefix}indicator_link"/>
       <!-- Plasserer indikatoren til å stikke ut fra disken (langs x-aksen) -->
-      <origin xyz="${disk_radius} 0 0" rpy="0 0 0"/>
+      <origin xyz="${disk_radius-0.012} 0 0.005" rpy="0 0 0"/>
     </joint>
   </xacro:macro>
