Commit message: Alt funka

File: src/qube_bringup/urdf/controlled_qube.urdf.xacro (robot description, xacro)
@@ -3,5 +3,5 @@
   <!-- Definer argument for makroer -->
   <xacro:arg name="baud_rate" default="115200"/>
-  <xacro:arg name="device" default="/dev/ttyUSB0"/>
+  <xacro:arg name="device" default="/dev/ttyACM0"/>
   <xacro:arg name="simulation" default="false"/>
   <!-- Inkluder makrofila frå qube_description og qube_driver -->

File: src/qube_description/urdf/qube.macro.xacro (robot description, xacro)
@@ -53,5 +53,5 @@
     </joint>
     <!-- Revolute joint: disken spinner i forhold til boksen -->
-    <joint name="${prefix}disk_joint" type="revolute">
+    <joint name="${prefix}motor_joint" type="revolute">
       <parent link="${prefix}stator_link"/>
       <child link="${prefix}rotor_link"/>
